File: electronics/right/electronics.kicad_sch (KiCad schematic)
At the start: 85 parts, among them J1 USB_C_Receptacle_USB2.0, J2 Molex_781710002, SW1 CPG135001S30, SW10 CPG135001S30, SW11 CPG135001S30, SW12 CPG135001S30, SW13 CPG135001S30, SW14 CPG135001S30, SW15 CPG135001S30, SW16 CPG135001S30, SW17 CPG135001S30, SW18 CPG135001S30, SW19 CPG135001S30, SW2 CPG135001S30, SW20 CPG135001S30, SW21 CPG135001S30, SW22 EVQPUC02K, SW3 CPG135001S30, SW4 CPG135001S30, SW5 CPG135001S30, SW6 CPG135001S30, SW7 CPG135001S30, SW8 CPG135001S30, SW9 CPG135001S30, U1 nRF52840, U2 ESDR0502NMUTAG, U3 BQ24075RGT, Y1 32.768 kHz, Y2 32MHz

Commit message: Fix incorrect manufacturer part numbers.
Parts:
- C19: Digikey 1276-1595-1-ND -> (none); JLC Part C1550 -> (none); LCSC Part C371977 -> (none); Manufacturer Part CL05C010CB5NNNC -> CL05C1R2CB5NNNC
- C4: Digikey 1276-6720-1-ND -> (none); JLC Part C1525 -> C14442; LCSC Part C1525 -> C14442; Manufacturer Part CL05B104KA5NNNC -> CL05B102KB5NNNC
- L4: JLC Part C14033 -> C136249; LCSC Part C76775 -> C136249; Manufacturer Part MLG1005S3N9BT000 -> MLG1005S2N2ST000
- L5: JLC Part C14033 -> C275292; LCSC Part C76775 -> C275292; Manufacturer Part MLG1005S3N9BT000 -> MLG1005S4N7CT000
- R6: JLC Part C25744 -> C138033; LCSC Part C60490 -> C138033; Manufacturer Part RC0402FR-0710KL -> RC0402FR-071ML
- R7, R8: JLC Part C25744 -> C105872; LCSC Part C60490 -> C105872; Manufacturer Part RC0402FR-0710KL -> RC0402FR-075K1L
Changed lines of the file:
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@@
       (effects (font (size 1.27 1.27)) hide)
     )
-    (property "LCSC Part" "C371977" (at 68.58 171.45 0)
+    (property "LCSC Part" "" (at 68.58 171.45 0)
       (effects (font (size 1.27 1.27)) hide)
     )
-    (property "Digikey" "1276-1595-1-ND" (at 68.58 171.45 0)
+    (property "Manufacturer Part" "CL05C1R2CB5NNNC" (at 68.58 171.45 0)
       (effects (font (size 1.27 1.27)) hide)
     )
-    (property "Manufacturer Part" "CL05C010CB5NNNC" (at 68.58 171.45 0)
-      (effects (font (size 1.27 1.27)) hide)
-    )
-    (property "JLC Part" "C1550" (at 68.58 171.45 0)
+    (property "JLC Part" "" (at 68.58 171.45 0)
       (effects (font (size 1.27 1.27)) hide)
     )
@@
       (effects (font (size 1.27 1.27)) hide)
     )
-    (property "LCSC Part" "C60490" (at 164.211 244.856 0)
+    (property "LCSC Part" "C138033" (at 164.211 244.856 0)
       (effects (font (size 1.27 1.27)) hide)
     )
-    (property "Manufacturer Part" "RC0402FR-0710KL" (at 164.211 244.856 0)
+    (property "Manufacturer Part" "RC0402FR-071ML " (at 164.211 244.856 0)
       (effects (font (size 1.27 1.27)) hide)
     )
-    (property "JLC Part" "C25744" (at 164.211 244.856 0)
+    (property "JLC Part" "C138033" (at 164.211 244.856 0)
       (effects (font (size 1.27 1.27)) hide)
     )
@@
       (effects (font (size 1.27 1.27)) hide)
     )
-    (property "LCSC Part" "C76775" (at 60.96 167.64 0)
+    (property "LCSC Part" "C136249" (at 60.96 167.64 0)
       (effects (font (size 1.27 1.27)) hide)
     )
-    (property "Manufacturer Part" "MLG1005S3N9BT000" (at 60.96 167.64 0)
+    (property "Manufacturer Part" "MLG1005S2N2ST000" (at 60.96 167.64 0)
       (effects (font (size 1.27 1.27)) hide)
     )
-    (property "JLC Part" "C14033" (at 60.96 167.64 0)
+    (property "JLC Part" "C136249" (at 60.96 167.64 0)
       (effects (font (size 1.27 1.27)) hide)
     )
@@
       (effects (font (size 1.27 1.27)) hide)
     )
-    (property "LCSC Part" "C60490" (at 195.326 270.51 0)
+    (property "LCSC Part" "C105872" (at 195.326 270.51 0)
       (effects (font (size 1.27 1.27)) hide)
     )
-    (property "Manufacturer Part" "RC0402FR-0710KL" (at 195.326 270.51 0)
+    (property "Manufacturer Part" "RC0402FR-075K1L " (at 195.326 270.51 0)
       (effects (font (size 1.27 1.27)) hide)
     )
-    (property "JLC Part" "C25744" (at 195.326 270.51 0)
+    (property "JLC Part" "C105872" (at 195.326 270.51 0)
       (effects (font (size 1.27 1.27)) hide)
     )
@@
       (effects (font (size 1.27 1.27)) hide)
     )
-    (property "LCSC Part" "C60490" (at 197.866 270.51 0)
+    (property "LCSC Part" "C105872" (at 197.866 270.51 0)
       (effects (font (size 1.27 1.27)) hide)
     )
-    (property "Manufacturer Part" "RC0402FR-0710KL" (at 197.866 270.51 0)
+    (property "Manufacturer Part" "RC0402FR-075K1L " (at 197.866 270.51 0)
       (effects (font (size 1.27 1.27)) hide)
     )
-    (property "JLC Part" "C25744" (at 197.866 270.51 0)
+    (property "JLC Part" "C105872" (at 197.866 270.51 0)
       (effects (font (size 1.27 1.27)) hide)
     )
@@
       (effects (font (size 1.27 1.27)) hide)
     )
-    (property "LCSC Part" "C1525" (at 101.6 123.19 0)
-      (effects (font (size 1.27 1.27)) hide)
-    )
-    (property "Digikey" "1276-6720-1-ND" (at 101.6 123.19 0)
+    (property "LCSC Part" "C14442" (at 101.6 123.19 0)
       (effects (font (size 1.27 1.27)) hide)
     )
-    (property "Manufacturer Part" "CL05B104KA5NNNC" (at 101.6 123.19 0)
+    (property "Manufacturer Part" "CL05B102KB5NNNC" (at 101.6 123.19 0)
       (effects (font (size 1.27 1.27)) hide)
     )
-    (property "JLC Part" "C1525" (at 101.6 123.19 0)
+    (property "JLC Part" "C14442" (at 101.6 123.19 0)
       (effects (font (size 1.27 1.27)) hide)
     )
@@
       (effects (font (size 1.27 1.27)) hide)
     )
-    (property "LCSC Part" "C76775" (at 73.66 167.64 0)
+    (property "LCSC Part" "C275292" (at 73.66 167.64 0)
       (effects (font (size 1.27 1.27)) hide)
     )
-    (property "Manufacturer Part" "MLG1005S3N9BT000" (at 73.66 167.64 0)
+    (property "Manufacturer Part" "MLG1005S4N7CT000" (at 73.66 167.64 0)
       (effects (font (size 1.27 1.27)) hide)
     )
-    (property "JLC Part" "C14033" (at 73.66 167.64 0)
+    (property "JLC Part" "C275292" (at 73.66 167.64 0)
       (effects (font (size 1.27 1.27)) hide)
     )
